File: ChargePCB/ChargePCB.kicad_pcb (KiCad board)
At the start: 2 copper layers, 80.2 x 37.1 mm, 38 parts, among them J1 Sol+, J2 Sol-, J3 USB_A, SW1 SW_SPDT, U1 LT3652, U2 S-8261, U3 DMG6968UDM, U4 RT4812

Commit message: changed silkscreen to say new repository
Other:
- board text added: "https://github.com/cosgais/Solar-Charger"
- board text removed: "https://github.com/T1gerc1aw/Solar-Charger"
Changed lines of the file:
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@@
       (net 3 GND))
   )
-  (gr_text https://github.com/T1gerc1aw/Solar-Charger (at 157 84.1) (layer B.SilkS)
+  (gr_text https://github.com/cosgais/Solar-Charger (at 157 84.1) (layer B.SilkS)
     (effects (font (size 1 1) (thickness 0.15)) (justify mirror))
   )
