File: ChargePCB/ChargePCB.kicad_pcb (KiCad board)
At the start: 2 copper layers, 80.2 x 37.1 mm, 38 parts, among them J1 Sol+, J2 Sol-, J3 USB_A, SW1 SW_SPDT, U1 LT3652, U2 S-8261, U3 DMG6968UDM, U4 RT4812

Commit message: Fixing USB polarity, Lipo Protection, and 1.5uH footprint error
Parts:
- J1: value Sol+ -> Conn_01x01_Male
- J2: value Sol- -> Conn_01x01_Male
- L2: footprint Inductor_SMD:L_0805_2012Metric -> Inductor_SMD:L_Bourns-SRN6028
- moved C6 2.18 mm to (139.4, 100.7)
- moved TP1 1.43 mm to (136.3, 108.1)
- moved L2 1.28 mm to (133.7, 102.5)
- turned U3 to 0 degrees
Connections:
- J3 pad 1: Net-(C8-Pad1) -> GND
- J3 pad 4: GND -> Net-(C8-Pad1)
- U3 pad 1: Net-(U2-Pad3) -> Bat-
- U3 pad 3: Net-(U2-Pad1) -> GND
- U3 pad 4: Bat- -> Net-(U2-Pad3)
- U3 pad 6: GND -> Net-(U2-Pad1)
Routing:
- net Net-(C8-Pad1): track 38.7 -> 44.5 mm
- net Net-(C1-Pad1): track 41.3 -> 44.7 mm
- net Net-(L2-Pad2): track 0.00 -> 2.29 mm
- net GND: track 71.0 -> 72.2 mm
